Commit message: mapa levine

File: description/robot_core.xacro (robot description, xacro)
@@ -36,5 +36,5 @@
             <origin xyz="0.12 0 0.05"/>
             <geometry>
-                <box size="0.24 0.20 0.10"/>
+                <box size="0.24 0.16 0.10"/>
             </geometry>
             <material name="white"/>

Commit message: mapeo de la pista levine

File: description/robot_core.xacro (robot description, xacro)
@@ -82,6 +82,6 @@
         <parent link="base_link"/>
         <child link="right_wheel"/>
-        <origin xyz="0 -0.10 0" rpy="${pi/2} 0 0"/>
-        <axis xyz="0 0 -1"/>
+        <origin xyz="0 -0.10 0" rpy="-${pi/2} 0 0"/>
+        <axis xyz="0 0 1"/>
     </joint>
     <link name="right_wheel">
